Commit message: Working looping with simple obstacle avoidance of wall bot

File: wall_bot_ws/src/wall_bot_description/urdf/wall_bot.urdf.xacro (robot description, xacro)
@@ -6,10 +6,10 @@
   <!-- Scale the original wall bot down so its footprint is close to LazyGo. -->
   <xacro:property name="model_scale" value="0.39"/>
-  <xacro:property name="base_length" value="${0.45 * model_scale}"/>
-  <xacro:property name="base_width"  value="${0.30 * model_scale}"/>
+  <xacro:property name="base_length" value="${0.40 * model_scale}"/>
+  <xacro:property name="base_width"  value="${0.25 * model_scale}"/>
   <xacro:property name="base_height" value="${0.12 * model_scale}"/>
   <xacro:property name="wheel_radius" value="${0.065 * model_scale}"/>
   <xacro:property name="wheel_width"  value="${0.035 * model_scale}"/>
-  <xacro:property name="wheel_separation" value="${0.32 * model_scale}"/>
+  <xacro:property name="wheel_separation" value="${0.34 * model_scale}"/>
   <xacro:property name="wheel_diameter" value="${0.13 * model_scale}"/>
   <xacro:property name="base_origin_z" value="${0.12 * model_scale}"/>
@@ -18,14 +18,12 @@
   <xacro:property name="wheel_marker_width" value="${0.002 * model_scale}"/>
   <xacro:property name="wheel_marker_height" value="${0.018 * model_scale}"/>
-  <xacro:property name="caster_radius" value="${0.035 * model_scale}"/>
-  <xacro:property name="caster_x_offset" value="${-0.16 * model_scale}"/>
   <xacro:property name="laser_radius" value="${0.055 * model_scale}"/>
   <xacro:property name="laser_length" value="${0.04 * model_scale}"/>
-  <xacro:property name="laser_x_offset" value="${-0.12 * model_scale}"/>
-  <xacro:property name="laser_z_offset" value="${0.22 * model_scale}"/>
-  <xacro:property name="camera_x_offset" value="0.06"/>
+  <xacro:property name="laser_x_offset" value="${0.1}"/>
+  <xacro:property name="laser_z_offset" value="${0.20 * model_scale}"/>
+  <xacro:property name="camera_x_offset" value="0.11"/>
   <xacro:property name="camera_y_offset" value="0.0"/>
   <xacro:property name="camera_z_offset" value="0.10"/>
-  <xacro:property name="camera_pitch" value="0.3"/>
+  <xacro:property name="camera_pitch" value="0.1"/>
   <!-- ========================= -->
   <!-- Materials -->
@@ -44,33 +42,8 @@
   </material>
   <!-- ========================= -->
-  <!-- Base link -->
-  <!-- ========================= -->
-  <link name="base_link">
-    <visual>
-      <origin xyz="0 0 ${base_origin_z}" rpy="0 0 0"/>
-      <geometry>
-        <box size="${base_length} ${base_width} ${base_height}"/>
-      </geometry>
-      <material name="orange"/>
-    </visual>
-    <collision>
-      <origin xyz="0 0 ${base_origin_z}" rpy="0 0 0"/>
-      <geometry>
-        <box size="${base_length} ${base_width} ${base_height}"/>
-      </geometry>
-    </collision>
-    <inertial>
-      <origin xyz="0 0 ${base_origin_z}" rpy="0 0 0"/>
-      <mass value="2.0"/>
-      <inertia
-        ixx="0.03" ixy="0.0" ixz="0.0"
-        iyy="0.03" iyz="0.0"
-        izz="0.04"/>
-    </inertial>
-  </link>
-  <!-- ========================= -->
-  <!-- Left wheel -->
-  <!-- ========================= -->
-  <link name="left_wheel_link">
+  <!-- Wheel macro -->
+  <!-- ========================= -->
+<xacro:macro name="wheel_link" params="name">
+  <link name="${name}">
     <visual>
       <origin xyz="0 0 0" rpy="1.5708 0 0"/>
@@ -94,12 +67,77 @@
     </inertial>
   </link>
-  <joint name="left_wheel_joint" type="continuous">
+</xacro:macro>
+<xacro:wheel_link name="rear_left_wheel_link"/>
+<xacro:wheel_link name="rear_right_wheel_link"/>
+<xacro:wheel_link name="front_left_wheel_link"/>
+<xacro:wheel_link name="front_right_wheel_link"/>
+  <!-- ========================= -->
+  <!-- Base link -->
+  <!-- ========================= -->
+  <link name="base_link">
+    <visual>
+      <origin xyz="0 0 ${base_origin_z}" rpy="0 0 0"/>
+      <geometry>
+        <box size="${base_length} ${base_width} ${base_height}"/>
+      </geometry>
+      <material name="orange"/>
+    </visual>
+    <collision>
+      <origin xyz="0 0 ${base_origin_z}" rpy="0 0 0"/>
+      <geometry>
+        <box size="${base_length} ${base_width} ${base_height}"/>
+      </geometry>
+    </collision>
+    <inertial>
+      <origin xyz="0 0 ${base_origin_z}" rpy="0 0 0"/>
+      <mass value="2.0"/>
+      <inertia
+        ixx="0.03" ixy="0.0" ixz="0.0"
+        iyy="0.03" iyz="0.0"
+        izz="0.04"/>
+    </inertial>
+  </link>
+  <!-- ========================= -->
+  <!--Front box link -->
+  <!-- ========================= -->
+    <link name="front_box_link">
+    <visual>
+      <origin xyz="0 0 ${base_origin_z}" rpy="0 0 0"/>
+      <geometry>
+        <box size="${base_length/2} ${base_width/2.2} ${base_height}"/>
+      </geometry>
+      <material name="orange"/>
+    </visual>
+    <collision>
+      <origin xyz="0 0 ${base_origin_z}" rpy="0 0 0"/>
+      <geometry>
+         <box size="${base_length/2} ${base_width/2} ${base_height/2}"/>
+      </geometry>
+    </collision>
+    <inertial>
+      <origin xyz="0 0 ${base_origin_z}" rpy="0 0 0"/>
+      <mass value="2.0"/>
+      <inertia
+        ixx="0.03" ixy="0.0" ixz="0.0"
+        iyy="0.03" iyz="0.0"
+        izz="0.04"/>
+    </inertial>
+  </link>
+    <joint name="front_box_base_link_joint" type="fixed">
     <parent link="base_link"/>
-    <child link="left_wheel_link"/>
-    <origin xyz="${wheel_x_offset} ${wheel_separation/2} ${wheel_radius}" rpy="0 0 0"/>
+    <child link="front_box_link"/>
+    <origin xyz="${base_length/2} 0 0" rpy="0 0 0"/>
+  </joint>
+  <!-- ========================= -->
+  <!--Rear Left wheel -->
+  <!-- ========================= -->
+  <joint name="rear_left_wheel_joint" type="continuous">
+    <parent link="base_link"/>
+    <child link="rear_left_wheel_link"/>
+    <origin xyz="-${wheel_x_offset} ${wheel_separation/2} ${wheel_radius}" rpy="0 0 0"/>
     <axis xyz="0 1 0"/>
   </joint>
   <!-- Left wheel rotation marker -->
-<link name="left_wheel_marker_link">
+<link name="rear_left_wheel_marker_link">
   <visual>
     <origin xyz="0 0 0" rpy="0 0 0"/>
@@ -110,42 +148,20 @@
   </visual>
 </link>
-<joint name="left_wheel_marker_joint" type="fixed">
-  <parent link="left_wheel_link"/>
-  <child link="left_wheel_marker_link"/>
+<joint name="rear_left_wheel_marker_joint" type="fixed">
+  <parent link="rear_left_wheel_link"/>
+  <child link="rear_left_wheel_marker_link"/>
   <origin xyz="${wheel_radius*0.65} ${wheel_width/2 } 0" rpy="0 0 0"/>
 </joint>
   <!-- ========================= -->
-  <!-- Right wheel -->
-  <!-- ========================= -->
-  <link name="right_wheel_link">
-    <visual>
-      <origin xyz="0 0 0" rpy="1.5708 0 0"/>
-      <geometry>
-        <cylinder radius="${wheel_radius}" length="${wheel_width}"/>
-      </geometry>
-      <material name="black"/>
-    </visual>
-    <collision>
-      <origin xyz="0 0 0" rpy="1.5708 0 0"/>
-      <geometry>
-        <cylinder radius="${wheel_radius}" length="${wheel_width}"/>
-      </geometry>
-    </collision>
-    <inertial>
-      <mass value="0.2"/>
-      <inertia
-        ixx="0.001" ixy="0.0" ixz="0.0"
-        iyy="0.001" iyz="0.0"
-        izz="0.001"/>
-    </inertial>
-  </link>
-  <joint name="right_wheel_joint" type="continuous">
+  <!-- Rear Right wheel -->
+  <!-- ========================= -->
+  <joint name="rear_right_wheel_joint" type="continuous">
     <parent link="base_link"/>
-    <child link="right_wheel_link"/>
-    <origin xyz="${wheel_x_offset} -${wheel_separation/2} ${wheel_radius}" rpy="0 0 0"/>
+    <child link="rear_right_wheel_link"/>
+    <origin xyz="-${wheel_x_offset} -${wheel_separation/2} ${wheel_radius}" rpy="0 0 0"/>
     <axis xyz="0 1 0"/>
   </joint>
-  <!-- Right wheel rotation marker -->
-<link name="right_wheel_marker_link">
+  <!-- Rear Right wheel rotation marker -->
+<link name="rear_right_wheel_marker_link">
   <visual>
     <origin xyz="0 0 0" rpy="0 0 0"/>
@@ -156,39 +172,115 @@
   </visual>
 </link>
-<joint name="right_wheel_marker_joint" type="fixed">
-  <parent link="right_wheel_link"/>
-  <child link="right_wheel_marker_link"/>
+<joint name="rear_right_wheel_marker_joint" type="fixed">
+  <parent link="rear_right_wheel_link"/>
+  <child link="rear_right_wheel_marker_link"/>
   <origin xyz="${wheel_radius*0.65} -${wheel_width/2} 0" rpy="0 0 0"/>
 </joint>
   <!-- ========================= -->
-  <!-- Caster wheel -->
-  <!-- ========================= -->
-  <link name="caster_link">
-    <visual>
+  <!-- Front Left Wheel -->
+  <!-- ========================= -->
+<link name = "front_left_steer_link">
+ <visual>
       <origin xyz="0 0 0" rpy="0 0 0"/>
       <geometry>
-        <sphere radius="${caster_radius}"/>
-      </geometry>
-      <material name="gray"/>
-    </visual>
-    <collision>
+        <box size="0.01 0.015 0.01"/>
+      </geometry>
+      <material name="white"/>
+    </visual>
+  <collision>
+    <origin xyz="0 0 0" rpy="0 0 0"/>
+    <geometry>
+      <box size="0.01 0.015 0.01"/>
+    </geometry>
+  </collision>
+  <inertial>
+    <mass value="0.02"/>
+    <inertia
+      ixx="0.00001" ixy="0.0" ixz="0.0"
+      iyy="0.00001" iyz="0.0"
+      izz="0.00001"/>
+  </inertial>
+</link>
+<joint name = "front_left_steer_joint" type="revolute">
+  <parent link="base_link"/>
+  <child link="front_left_steer_link"/>
+  <origin xyz="${base_length / 1.4} ${base_width/2.4} ${wheel_radius}" rpy="0 0 0"/>
+  <axis xyz="0 0 1"/>
+  <limit lower="-0.6" upper="0.6" effort="10.0" velocity="5.0" />
+</joint>
+  <joint name="front_left_wheel_joint" type="continuous">
+    <parent link="front_left_steer_link"/>
+    <child link="front_left_wheel_link"/>
+    <origin xyz="0 0 0" rpy="0 0 0"/>
+    <axis xyz="0 1 0"/>
+  </joint>
+    <!-- Front Left wheel rotation marker -->
+<link name="front_left_wheel_marker_link">
+  <visual>
+    <origin xyz="0 0 0" rpy="0 0 0"/>
+    <geometry>
+      <box size="${wheel_marker_length} ${wheel_marker_width} ${wheel_marker_height}"/>
+    </geometry>
+    <material name="white"/>
+  </visual>
+</link>
+<joint name="front_left_wheel_marker_joint" type="fixed">
+  <parent link="front_left_wheel_link"/>
+  <child link="front_left_wheel_marker_link"/>
+  <origin xyz="${wheel_radius*0.65} ${wheel_width/2 } 0" rpy="0 0 0"/>
+</joint>
+  <!-- ========================= -->
+  <!-- Front Right Wheel -->
+  <!-- ========================= -->
+<link name = "front_right_steer_link">
+ <visual>
       <origin xyz="0 0 0" rpy="0 0 0"/>
       <geometry>
-        <sphere radius="${caster_radius}"/>
-      </geometry>
-    </collision>
-    <inertial>
-      <mass value="0.05"/>
-      <inertia
-        ixx="0.0001" ixy="0.0" ixz="0.0"
-        iyy="0.0001" iyz="0.0"
-        izz="0.0001"/>
-    </inertial>
-  </link>
-  <joint name="caster_joint" type="fixed">
-    <parent link="base_link"/>
-    <child link="caster_link"/>
-    <origin xyz="${caster_x_offset} 0 ${caster_radius}" rpy="0 0 0"/>
-  </joint>
+        <box size="0.01 0.015 0.01"/>
+      </geometry>
+      <material name="white"/>
+    </visual>
+  <collision>
+    <origin xyz="0 0 0" rpy="0 0 0"/>
+    <geometry>
+      <box size="0.01 0.015 0.01"/>
+    </geometry>
+  </collision>
+  <inertial>
+    <mass value="0.02"/>
+    <inertia
+      ixx="0.00001" ixy="0.0" ixz="0.0"
+      iyy="0.00001" iyz="0.0"
+      izz="0.00001"/>
+  </inertial>
+</link>
+<joint name = "front_right_steer_joint" type="revolute">
+  <parent link="base_link"/>
+  <child link="front_right_steer_link"/>
+  <origin xyz="${base_length / 1.4} -${base_width/2.4} ${wheel_radius}" rpy="0 0 0"/>
+  <axis xyz="0 0 1"/>
+  <limit lower="-0.6" upper="0.6" effort="10.0" velocity="5.0" />
+</joint>
+  <joint name="front_right_wheel_joint" type="continuous">
+    <parent link="front_right_steer_link"/>
+    <child link="front_right_wheel_link"/>
+    <origin xyz="0 0 0" rpy="0 0 0"/>
+    <axis xyz="0 1 0"/>
+  </joint>
+    <!-- Front Left wheel rotation marker -->
+<link name="front_right_wheel_marker_link">
+  <visual>
+    <origin xyz="0 0 0" rpy="0 0 0"/>
+    <geometry>
+      <box size="${wheel_marker_length} ${wheel_marker_width} ${wheel_marker_height}"/>
+    </geometry>
+    <material name="white"/>
+  </visual>
+</link>
+<joint name="front_right_wheel_marker_joint" type="fixed">
+  <parent link="front_right_wheel_link"/>
+  <child link="front_right_wheel_marker_link"/>
+  <origin xyz="${wheel_radius*0.65} ${wheel_width/2 } 0" rpy="0 0 0"/>
+</joint>
   <!-- ========================= -->
   <!-- LiDAR -->
@@ -250,5 +342,14 @@
     <material>Gazebo/Orange</material>
   </gazebo>
-  <gazebo reference="left_wheel_link">
+  <gazebo reference="front_box_link">
+    <material>Gazebo/Orange</material>
+  </gazebo>
+  <gazebo reference="front_left_steer_link">
+    <material>Gazebo/Grey</material>
+  </gazebo>
+  <gazebo reference="front_right_steer_link">
+    <material>Gazebo/Grey</material>
+  </gazebo>
+  <gazebo reference="front_left_wheel_link">
     <material>Gazebo/Black</material>
     <mu1>20.0</mu1>
@@ -257,5 +358,5 @@
     <slip2>0.0</slip2>
   </gazebo>
-  <gazebo reference="right_wheel_link">
+  <gazebo reference="front_right_wheel_link">
     <material>Gazebo/Black</material>
     <mu1>20.0</mu1>
@@ -264,42 +365,18 @@
     <slip2>0.0</slip2>
   </gazebo>
-  <!-- Keep the caster easy to skid so it does not fight differential turns. -->
-  <gazebo reference="caster_link">
-    <material>Gazebo/Grey</material>
-    <mu1>0.05</mu1>
-    <mu2>0.05</mu2>
-    <slip1>1.0</slip1>
-    <slip2>1.0</slip2>
-  </gazebo>
-  <!-- ========================= -->
-  <!-- Differential drive plugin -->
-  <!-- ========================= -->
-  <gazebo>
-    <plugin name="gazebo_ros_diff_drive" filename="libgazebo_ros_diff_drive.so">
-      <update_rate>100</update_rate>
-      <left_joint>left_wheel_joint</left_joint>
-      <right_joint>right_wheel_joint</right_joint>
-      <wheel_separation>${wheel_separation}</wheel_separation>
-      <wheel_diameter>${wheel_diameter}</wheel_diameter>
-      <max_wheel_torque>30</max_wheel_torque>
-      <max_wheel_acceleration>30.0</max_wheel_acceleration>
-      <command_topic>cmd_vel</command_topic>
-      <odometry_topic>odom</odometry_topic>
-      <odometry_frame>odom</odometry_frame>
-      <robot_base_frame>base_link</robot_base_frame>
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